Commit message: Add VHACD collision meshes, collision visualization, and panda-gym integration
- Replace raw-mesh collision geometry with VHACD convex decompositions
  (urdf/meshes/collision/*.obj; base 8 hulls, fingers 4 hulls each),
  regenerable via scripts/simplify_meshes.py + tools/TestVHACD.exe
- Add collision_visual.py: green ghost overlay of URDF collision meshes
  in PyBullet, V key cycles visual/collision display in all demos
- Add keyboard_control_franka.py: gripper mounted on a Franka Panda
  (URDF generated by scripts/make_panda_with_gripper.py)
- Add panda_force_gripper.py: panda-gym robot class + Reach and
  PickAndPlace envs for the mounted gripper
- Add keyboard_pick_and_place.py: keyboard-driven pick and place in the
  panda-gym scene with 6-DOF end-effector control (IK position + tool
  euler angles)

File: urdf/force_control_gripper.urdf (robot description, URDF)
Before this commit: robot force_control_gripper, 3 links, 2 joints
Links:
- link base-1: geometry collision mesh filename=meshes/collision/base-1_collision.obj scale=0.001 0.001 0.001; visual mesh filename=meshes/base-1.stl scale=0.001 0.001 0.001
- link left_figure: geometry collision mesh filename=meshes/collision/left_figure_collision.obj scale=0.001 0.001 0.001; visual mesh filename=meshes/left_figure.stl scale=0.001 0.001 0.001
- link right_figure: geometry collision mesh filename=meshes/collision/right_figure_collision.obj scale=0.001 0.001 0.001; visual mesh filename=meshes/right_figure.stl scale=0.001 0.001 0.001
